File: BlinkyBall.brd (EAGLE design)
At the start: 4 parts, among them IC3 TINY13-20SSU

Commit message: Fixups to board
Routing:
- net S$2: track 2.79 -> 5.08 mm
- net S$10: track 0.00 -> 1.59 mm
- net S$7: track 7.30 -> 8.41 mm
- net S$4: track 9.33 -> 8.29 mm
Other:
- board text added: "bb40"
- board text added: "data"
- board text added: "man"
- board text removed: "bb32"
Changed lines of the file:
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@@
 <plain>
 <circle x="8.41375" y="8.5725" radius="0.3175" width="0.4064" layer="1"/>
-<text x="18.89125" y="12.3825" size="1.778" layer="1" rot="R90">bb32</text>
+<text x="18.89125" y="12.3825" size="1.778" layer="1" rot="R90">bb40</text>
 <circle x="15.24" y="16.98625" radius="0.3175" width="0.4064" layer="16"/>
-<rectangle x1="7.62" y1="15.08125" x2="10.16" y2="17.62125" layer="16"/>
-<rectangle x1="11.58875" y1="5.715" x2="14.12875" y2="8.255" layer="16"/>
-<rectangle x1="13.6525" y1="16.1925" x2="16.66875" y2="17.78" layer="16"/>
-<rectangle x1="13.6525" y1="13.49375" x2="16.66875" y2="15.08125" layer="16"/>
+<rectangle x1="7.77875" y1="15.5575" x2="10.31875" y2="18.0975" layer="1"/>
+<rectangle x1="11.58875" y1="5.08" x2="14.12875" y2="7.62" layer="1"/>
+<rectangle x1="13.6525" y1="16.1925" x2="16.66875" y2="17.78" layer="1"/>
+<rectangle x1="13.6525" y1="13.49375" x2="16.66875" y2="15.08125" layer="1"/>
+<text x="17.30375" y="3.01625" size="1.778" layer="1" rot="R90">data</text>
+<text x="18.89125" y="3.01625" size="1.778" layer="1" rot="R90">man</text>
 </plain>
 <attributes>
@@
 <signal name="S$2">
 <wire x1="10.63625" y1="3.96875" x2="12.065" y2="3.96875" width="0.6096" layer="1"/>
-<wire x1="15.71625" y1="14.76375" x2="14.605" y2="13.97" width="0.6096" layer="16"/>
+<wire x1="16.35125" y1="14.76375" x2="16.35125" y2="11.1125" width="0.6096" layer="1"/>
 </signal>
 <signal name="S$3">
@@
 </signal>
 <signal name="S$4">
-<wire x1="2.69875" y1="10.31875" x2="2.69875" y2="14.12875" width="0.4064" layer="16"/>
-<wire x1="2.69875" y1="14.12875" x2="4.445" y2="14.44625" width="0.4064" layer="16"/>
-<wire x1="4.445" y1="14.44625" x2="6.0325" y2="14.44625" width="0.4064" layer="16"/>
-<wire x1="6.0325" y1="14.44625" x2="8.09625" y2="13.81125" width="0.4064" layer="16"/>
+<wire x1="3.33375" y1="11.43" x2="3.33375" y2="14.2875" width="0.6096" layer="1"/>
+<wire x1="3.33375" y1="14.2875" x2="3.65125" y2="14.44625" width="0.4064" layer="1"/>
+<wire x1="3.65125" y1="14.44625" x2="8.09625" y2="14.44625" width="0.6096" layer="1"/>
+<wire x1="8.09625" y1="14.44625" x2="8.09625" y2="13.81125" width="0.6096" layer="1"/>
 </signal>
 <signal name="S$5">
-<wire x1="2.8575" y1="16.51" x2="2.8575" y2="18.25625" width="0.4064" layer="16"/>
-<wire x1="2.8575" y1="18.25625" x2="6.6675" y2="18.25625" width="0.4064" layer="16"/>
-<wire x1="6.6675" y1="18.25625" x2="6.6675" y2="17.145" width="0.4064" layer="16"/>
+<wire x1="2.8575" y1="16.51" x2="2.8575" y2="18.25625" width="0.4064" layer="1"/>
+<wire x1="2.8575" y1="18.25625" x2="6.6675" y2="18.25625" width="0.4064" layer="1"/>
+<wire x1="6.6675" y1="18.25625" x2="6.6675" y2="17.145" width="0.4064" layer="1"/>
 </signal>
 <signal name="S$6">
-<wire x1="5.08" y1="15.71625" x2="8.41375" y2="15.71625" width="0.4064" layer="16"/>
+<wire x1="5.08" y1="15.71625" x2="7.9375" y2="15.71625" width="0.4064" layer="1"/>
 </signal>
 <signal name="S$7">
-<wire x1="6.6675" y1="12.85875" x2="6.6675" y2="6.985" width="0.4064" layer="16"/>
-<wire x1="6.6675" y1="6.985" x2="8.09625" y2="6.985" width="0.4064" layer="16"/>
+<wire x1="6.6675" y1="12.85875" x2="6.6675" y2="6.0325" width="0.6096" layer="1"/>
+<wire x1="6.6675" y1="6.0325" x2="8.255" y2="6.0325" width="0.6096" layer="1"/>
 </signal>
 <signal name="S$8">
-<wire x1="12.065" y1="11.90625" x2="15.08125" y2="8.5725" width="0.6096" layer="16"/>
-<wire x1="15.08125" y1="8.5725" x2="15.08125" y2="2.54" width="0.6096" layer="16"/>
-<wire x1="15.08125" y1="2.54" x2="10.63625" y2="2.54" width="0.6096" layer="16"/>
+<wire x1="12.065" y1="11.90625" x2="15.08125" y2="8.5725" width="0.6096" layer="1"/>
+<wire x1="15.08125" y1="8.5725" x2="15.08125" y2="2.54" width="0.6096" layer="1"/>
+<wire x1="15.08125" y1="2.54" x2="10.63625" y2="2.54" width="0.6096" layer="1"/>
 </signal>
 <signal name="S$9">
-<wire x1="5.08" y1="15.71625" x2="5.08" y2="16.98625" width="0.6096" layer="16"/>
+<wire x1="5.08" y1="15.875" x2="5.08" y2="16.98625" width="0.6096" layer="1"/>
+</signal>
+<signal name="S$10">
+<wire x1="4.28625" y1="7.14375" x2="4.28625" y2="8.73125" width="0.6096" layer="1"/>
 </signal>
 </signals>
